File: bcard/bcard.kicad_pcb (KiCad board)
At the start: 2 copper layers, 82 x 50 mm, 2 parts

Commit message: 0: fixed prod
Parts:
- moved G*** 0.61 mm to (132.9, 85.1)
Routing:
- net (no net): vias 0 -> 8
